File: schematics/kiCad/blinky-cube.kicad_sch (KiCad schematic)
At the start: 25 parts, among them J1 Screw_Terminal_01x03, J2 Screw_Terminal_01x03, J3 Screw_Terminal_01x03, SW1 SW_Push, U1 Pico, U2 LM4040LP-3

Commit message: thru hole
Parts:
- removed C2, C6: 1uF, Capacitor_SMD:C_1206_3216Metric_Pad1.33x1.80mm_HandSolder, symbol Device:C
- removed J1, J2, J3: Screw_Terminal_01x03, TerminalBlock:TerminalBlock_bornier-3_P5.08mm, symbol Connector:Screw_Terminal_01x03
- removed R3: 220, Resistor_SMD:R_1206_3216Metric_Pad1.30x1.75mm_HandSolder, symbol Device:R
- removed U2: LM4040LP-3, Package_TO_SOT_THT:TO-92_Inline, symbol Reference_Voltage:LM4040LP-3
- added J2: Barrel_Jack_Switch, Connector_BarrelJack:BarrelJack_Horizontal, symbol Connector:Barrel_Jack_Switch
- added J4, J5: Screw_Terminal_01x02, TerminalBlock_Phoenix:TerminalBlock_Phoenix_MKDS-3-2-5.08_1x02_P5.08mm_Horizontal, symbol Connector:Screw_Terminal_01x02
- C1, C3, C4, C5: footprint Capacitor_SMD:C_1206_3216Metric_Pad1.33x1.80mm_HandSolder -> Capacitor_THT:C_Disc_D4.7mm_W2.5mm_P5.00mm
- R1, R10, R11, R12, R2, R4, R5, R6, R7, R8, R9: footprint Resistor_SMD:R_1206_3216Metric_Pad1.30x1.75mm_HandSolder -> Resistor_THT:R_Axial_DIN0207_L6.3mm_D2.5mm_P7.62mm_Horizontal
Connections:
- net GND: now also J2.2, J4.2 (Pin_2), J5.2 (Pin_2)
- net at C1.1: now also R4.2, R5.2, R6.2, U1.39 (VSYS), J2.1; no longer U1.40 (VBUS)
- net at C4.1, R5.1, R9.1: now also J4.1 (Pin_1)
- net at C5.1, R11.1, R6.1: now also J5.1 (Pin_1)
- no-connect marks 24 -> 29
